Commit message: feat: update models for fixed URDF upstream

File: assets/mirobot_v2.urdf.xacro (robot description, xacro)
@@ -4,5 +4,5 @@
     <xacro:property name="hw_interface" value="$(arg hw_interface)"/>
     <xacro:property name="prefix" value=""/>
-    <xacro:include filename="$(find Mirobot_V2_URDF_Files)/urdf/Mirobot_V2_URDF_Files.urdf"/>
+    <xacro:include filename="$(find mirobot_urdf)/urdf/mirobot_urdf.urdf" />
     <xacro:macro name="transmission" params="prefix joint_name hw_interface">
         <transmission name="${prefix}${joint_name}_trans">

File: assets/mirobot_v2.xml.xacro (robot description, xacro)
@@ -1,4 +1,4 @@
 <?xml version="1.0" encoding="utf-8"?>
-<mujoco model="Mirobot_V2" xmlns:xacro="http://www.ros.org/wiki/xacro">
+<mujoco model="mirobot_urdf"  xmlns:xacro="http://www.ros.org/wiki/xacro">
   <xacro:arg name="control_rate" default="500"/>
   <xacro:property name="control_rate"     value="$(arg control_rate)"/>
@@ -25,13 +25,14 @@
     </default>
   </default>
+  <statistic meansize="0.0683645" extent="0.410433" center="0.170127 0.0599294 0.136871" />
   <asset>
-    <mesh name="base_link_Collision" file="$(find Mirobot_V2_URDF_Files)/meshes/base_link.STL" />
-    <mesh name="link1_Collision"     file="$(find Mirobot_V2_URDF_Files)/meshes/link1.STL" />
-    <mesh name="link2_Collision"     file="$(find Mirobot_V2_URDF_Files)/meshes/link2.STL" />
-    <mesh name="link3_Collision"     file="$(find Mirobot_V2_URDF_Files)/meshes/link3.STL" />
-    <mesh name="link4_Collision"     file="$(find Mirobot_V2_URDF_Files)/meshes/link4.STL" />
-    <mesh name="link5_Collision"     file="$(find Mirobot_V2_URDF_Files)/meshes/link5.STL" />
-    <mesh name="link6_Collision"     file="$(find Mirobot_V2_URDF_Files)/meshes/link6.STL" />
-    <mesh name="link61"              file="$(find Mirobot_V2_URDF_Files)/meshes/link61.STL"/>
+    <mesh name="base_link_collision" file="$(find mirobot_urdf)/meshes/base_link_collision.STL" />
+    <mesh name="link1_collision"     file="$(find mirobot_urdf)/meshes/link1_collision.STL" />
+    <mesh name="link2_collision"     file="$(find mirobot_urdf)/meshes/link2_collision.STL" />
+    <mesh name="link3_collision"     file="$(find mirobot_urdf)/meshes/link3_collision.STL" />
+    <mesh name="link4_collision"     file="$(find mirobot_urdf)/meshes/link4_collision.STL" />
+    <mesh name="link5_collision"     file="$(find mirobot_urdf)/meshes/link5_collision.STL" />
+    <mesh name="link6_collision"     file="$(find mirobot_urdf)/meshes/link6_collision.STL" />
+    <mesh name="link61"              file="$(find mirobot_urdf)/meshes/link61.STL" />
   </asset>
   <worldbody>
@@ -39,28 +40,28 @@
     <body name="base" pos="0 0 0" gravcomp="1" childclass="robot">
       <body name="base_link" pos="0 0 0" gravcomp="1">
-        <inertial pos="0.061385 0.061385 0.029563" quat="0.5 0.5 -0.5 0.5" mass="0.83046" diaginertia="0.0018135 0.0012252 0.0012252" />
-        <geom type="mesh" rgba="0.47843 0.47843 0.47843 1" mesh="base_link_Collision" />
+        <inertial pos="0.061385 0.061385 0.0295631" quat="0.5 0.5 -0.5 0.5" mass="0.83046" diaginertia="0.00181346 0.00122515 0.00122515" />
+        <geom type="mesh" rgba="0.478431 0.478431 0.478431 1" mesh="base_link_collision" />
         <body name="link1" pos="0.061385 0.061385 0" gravcomp="1">
-          <inertial pos="0.013921 0.00013535 0.11689" quat="0.637898 0.301943 0.305954 0.63899" mass="0.10078" diaginertia="6.20703e-05 5.14972e-05 2.49376e-05" />
+          <inertial pos="0.0139209 0.000135347 0.11689" quat="0.637896 0.301947 0.305957 0.638989" mass="0.100784" diaginertia="6.20698e-05 5.14973e-05 2.49373e-05" />
           <joint name="Joint1" pos="0 0 0" axis="0 0 1" range="-1.919 2.792" />
-          <geom type="mesh" rgba="0.79216 0.81961 0.93333 1" mesh="link1_Collision" />
-          <body name="link2" pos="0.02666 -0.010077 0.12699" gravcomp="1">
+          <geom type="mesh" rgba="0.792157 0.819608 0.933333 1" mesh="link1_collision" />
+          <body name="link2" pos="0.0266598 -0.0100773 0.126989" gravcomp="1">
             <inertial pos="-0.000147878 -0.0166549 0.0497584" quat="0.708147 0.000213996 6.89968e-05 0.706065" mass="0.132171" diaginertia="0.000225757 0.000214472 2.33029e-05" />
-            <joint name="Joint2" pos="0 0 0" axis="0.00289699 0.999996 0" range="-0.611 1.222" />
-            <geom type="mesh" rgba="1 0.6 0.247059 1" mesh="link2_Collision" />
-            <body name="link3" pos="-0.00013383 0 0.10356" gravcomp="1">
+            <joint name="Joint2" pos="0 0 0" axis="0.00289701 0.999996 0" range="-0.611 1.222" />
+            <geom type="mesh" rgba="1 0.6 0.247059 1" mesh="link2_collision" />
+            <body name="link3" pos="-0.000133826 0 0.103558" gravcomp="1">
               <inertial pos="0.015981 0.0217695 0.00460564" quat="0.00543631 0.61574 -0.00358634 0.787923" mass="0.0999859" diaginertia="0.000128775 0.000119394 2.89671e-05" />
-              <joint name="Joint3" pos="0 0 0" axis="0.00289699 0.999996 0" range="-2.094 1.047" />
-              <geom type="mesh" rgba="0.792157 0.819608 0.933333 1" mesh="link3_Collision" />
+              <joint name="Joint3" pos="0 0 0" axis="0.00289701 0.999996 0" range="-2.094 1.047" />
+              <geom type="mesh" rgba="0.792157 0.819608 0.933333 1" mesh="link3_collision" />
               <body name="link4" pos="0.11139 0.020972 0.019459" gravcomp="1">
                 <inertial pos="0.0397442 -0.000115496 -0.000190508" quat="-0.000509113 0.708816 -0.00253453 0.705389" mass="0.0455777" diaginertia="2.34679e-05 1.74414e-05 1.02362e-05" />
                 <joint name="Joint4" pos="0 0 0" axis="-0.999984 0.00289701 0.00481472" range="-3.142 3.142" />
-                <geom type="mesh" rgba="1 0.6 0.247059 1" mesh="link4_Collision" />
-                <body name="link5" pos="0.05775 -8.4329e-05 -0.019582" gravcomp="1">
-                  <inertial pos="-7.4482e-07 -5.0563e-05 0.011751" quat="0.999997 0.00215741 -2.85633e-05 -0.00145912" mass="0.014383" diaginertia="1.943e-06 1.83051e-06 1.09309e-06" />
-                  <joint name="Joint5" pos="0 0 0" axis="0.00291759 0.999987 0.00429129" range="-3.49 0.523" />
-                  <geom type="mesh" rgba="0.79216 0.81961 0.93333 1" mesh="link5_Collision" />
-                  <body name="link6" pos="0 6.822e-05 -0.016" quat="0.707105 0 0.707108 0" gravcomp="1">
-                    <joint name="Joint6" pos="0 0 0" axis="-0.999991 -0.0042638 -6.32701e-05" range="-6.283 6.283" />
+                <geom type="mesh" rgba="1 0.6 0.247059 1" mesh="link4_collision" />
+                <body name="link5" pos="0.057767 0.0061276 -0.00025103" quat="-3.67321e-06 1 0 0" gravcomp="1">
+                  <inertial pos="-1.78881e-05 0.00626251 0.00757976" quat="0.999997 0.00215724 2.85613e-05 0.00145901" mass="0.0143828" diaginertia="1.94302e-06 1.83053e-06 1.09304e-06" />
+                  <joint name="Joint5" pos="0 0 0" axis="0.00291759 -0.999987 -0.00429129" range="-3.49 0.523" />
+                  <geom type="mesh" rgba="0.792157 0.819608 0.933333 1" mesh="link5_collision" />
+                  <body name="link6" pos="-1.7143e-05 0.0062119 0.019331" quat="0.707105 -0.707108 0 0" gravcomp="1">
+                    <joint name="Joint6" pos="0 0 0" axis="-6.32701e-05 0.999991 0.0042638" range="-6.283 6.283" />
                     <geom type="cylinder" size="0.001 0.001" mass="0.001"/>
                   </body>
@@ -77,8 +78,8 @@
       <freejoint/>
       <body name="link6_compliant" gravcomp="0">
-        <inertial pos="-0.00022444 6.6311e-05 0.025902" quat="0.705615 0.00175116 0.00359626 0.708585" mass="0.041887" diaginertia="3.52612e-05 3.52048e-05 3.56617e-06" />
-        <geom type="mesh" rgba="1 1 1 1" mesh="link6_Collision" />
+        <inertial pos="0.020487 -0.017507 -0.00012792" quat="0.0273834 0.707513 -0.0298504 0.705538" mass="0.038132" diaginertia="2.62392e-05 2.61176e-05 3.39792e-06" />
+        <geom type="mesh" rgba="1 1 1 1" mesh="link6_collision" />
         <body name="link61" pos="0 0 0" gravcomp="0">
-          <inertial pos="-5.2733e-06 0.00018406 0.070942" quat="0.50063 0.499332 -0.499369 0.500667" mass="0.11219" diaginertia="1.5538e-05 1.0568e-05 1.0568e-05" />
+          <inertial pos="0.060943 -0.020995 -0.00024766" quat="0.999999 4.82219e-08 0.00129737 3.71689e-05" mass="0.11219" diaginertia="1.5538e-05 1.0568e-05 1.0568e-05" />
           <geom type="mesh" rgba="1 1 1 1" mesh="link61" />
           <site name="sensorsite"/>
